File: ALU_Tester.kicad_pcb (KiCad board)
At the start: 2 copper layers, 15 parts, among them J1 Conn_02x18_Odd_Even, J2 Conn_01x02, SW1 SW_SPST, U1 74LS181, U2 74LS181

Commit message: Upadate board
Update of board, fixed 24 pin ic size, adjusted board size.
Parts:
- U1, U2: footprint Package_DIP:DIP-24_W7.62mm_LongPads -> Package_DIP:DIP-24_W15.24mm_LongPads
- moved C1 39.6 mm to (145.3, 78.7)
- moved C2 38.1 mm to (117.9, 78.7)
- moved D1 12.4 mm to (154.7, 106.7)
- moved D2 12.4 mm to (154.7, 110.5)
- moved D3 12.4 mm to (164.8, 99.1)
- moved D4 12.4 mm to (152.1, 99.1)
- moved R3 12.4 mm to (162.3, 82.5)
- moved R4 12.4 mm to (154.7, 82.5)
- moved SW1 5.76 mm to (92.2, 110.5)
- moved U2 5.59 mm to (130.0, 82.5)
- moved J2 4.75 mm to (91.9, 100.3)
- moved R2 4.57 mm to (91.9, 78.7)
- moved R1 3.05 mm to (95.8, 78.7)
- moved U1 1.02 mm to (102.6, 82.5)
Routing:
- net D43: track 101.4 -> 55.9 mm
- net D37: track 58.8 -> 99.0 mm
- net GND: track 131.2 -> 165.3 mm
- net 5V: track 139.7 -> 106.5 mm
- net D47: track 55.5 -> 87.0 mm
- net D49: track 67.7 -> 89.5 mm
- net D46: track 58.2 -> 78.9 mm
- net D36: track 101.0 -> 80.3 mm
- net D48: track 63.8 -> 81.6 mm
- net D30: track 30.3 -> 44.7 mm
- net D35: track 93.0 -> 79.2 mm
- net D42: track 60.6 -> 72.3 mm
- net D25: track 43.8 -> 54.5 mm
- net D29: track 64.5 -> 74.3 mm, vias 1 -> 0
- net D23: track 36.2 -> 44.8 mm
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- added copper zone on B.Cu, net GND
Other:
- board text added: "ALU Tester Rev 2,"
